File: teensy_2026.kicad_sch (KiCad schematic)
At the start: 6 parts, among them J1 LED, U1 RASPBERRY_PI_PICO

Commit message: added linear actuator hall_effect
Parts:
- added J15: LinAct1, teensy:4pinJST, symbol Connector:Conn_01x04_Pin
- added J5: LinAct2, teensy:4pinJST, symbol Connector:Conn_01x04_Pin
Connections:
- net +5V: now also J15.3 (Pin_3), J5.3 (Pin_3)
- net GND: now also J15.4 (Pin_4), J5.4 (Pin_4)
- net LA1_HE1_in: now reaches U1.GP6
- net LA1_HE1_in: now also J15.1 (Pin_1)
- net LA1_HE2_in: now reaches U1.GP7
- net LA1_HE2_in: now also J15.2 (Pin_2)
- net LA2_HE1_in: now reaches U1.GP8
- net LA2_HE1_in: now also J5.1 (Pin_1)
- net LA2_HE2_in: now reaches U1.GP9
- net LA2_HE2_in: now also J5.2 (Pin_2)
